File: [02]Designs/KiCad Designs/463 term project.kicad_sch (KiCad schematic)
At the start: 142 parts, among them J1 Conn_01x02_Pin, J10 Conn_01x01_Pin, J11 Conn_01x01_Pin, J12 Conn_01x01_Pin, J13 Conn_01x01_Pin, J14 Conn_01x01_Pin, J15 Conn_01x01_Pin, J16 Conn_01x01_Pin, J17 Conn_01x01_Pin, J18 Conn_01x02_Pin, J19 Conn_01x02_Pin, J2 Screw_Terminal_01x01, J20 Conn_01x02_Pin, J21 Conn_01x02_Pin, J22 Conn_01x02_Pin, J23 Conn_01x02_Pin, J24 Conn_01x02_Pin, J25 Conn_01x02_Pin, J26 Conn_01x02_Pin, J3 Screw_Terminal_01x01, J4 Conn_01x03_Pin, J5 Screw_Terminal_01x01, J6 Screw_Terminal_01x01, J7 Conn_01x02_Pin, J8 Conn_01x01_Pin, J9 Conn_01x01_Pin, Q1 BC547, Q10 PJMH099N60EC, Q11 PJMH099N60EC, Q2 BC547, Q7 PJMH099N60EC, Q8 PJMH099N60EC, Q9 PJMH099N60EC, SW1 SW_Nidec_CAS-120A1, T2 Transformer, U1 6N135, U10 ADuM1200AR, U11 IR2110, U12 LM7805_TO220, U14 LM7815_TO220, U16 LD1117S33TR_SOT223, U17 LD1117S33TR_SOT223, U18 5 Button Module, U19 LM7812_TO220, U2 6N135, U20 LM7812_TO220, U3 74HC00, U4 IR2110, U5 IR2110, U6 ACS712xLCTR-30A, U8 ADuM1200AR, U9 ADuM1200AR

Commit message: [Design] Layout Finalized
Parts:
- added R18, R19: 0, Resistor_THT:R_Axial_DIN0207_L6.3mm_D2.5mm_P10.16mm_Horizontal, symbol Device:R
Connections:
- net GND: now also R18.2, R19.1
- net GNDD: now also R19.2
- net GNDPWR: now also R18.1
Changed lines of the file:
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@@
 	)
 	(junction
+		(at 50.8 83.82)
+		(diameter 0)
+		(color 0 0 0 0)
+	)
+	(junction
 		(at 167.64 267.97)
 		(diameter 0)
@@
 	(wire
 		(pts
+			(xy 59.69 83.82) (xy 59.69 87.63)
+		)
+		(stroke
+			(width 0)
+			(type default)
+		)
+	)
+	(wire
+		(pts
 			(xy 226.06 148.59) (xy 223.52 148.59)
 		)
@@
 	(wire
 		(pts
+			(xy 50.8 83.82) (xy 52.07 83.82)
+		)
+		(stroke
+			(width 0)
+			(type default)
+		)
+	)
+	(wire
+		(pts
 			(xy 139.7 175.26) (xy 163.83 175.26)
 		)
@@
 	(wire
 		(pts
+			(xy 49.53 83.82) (xy 50.8 83.82)
+		)
+		(stroke
+			(width 0)
+			(type default)
+		)
+	)
+	(wire
+		(pts
 			(xy 104.14 351.79) (xy 104.14 342.9)
 		)
@@
 	(symbol
 		(lib_id "power:GND")
-		(at 41.91 87.63 0)
+		(at 50.8 87.63 0)
+		(mirror y)
 		(unit 1)
 		(exclude_from_sim no)
@@
 		(fields_autoplaced yes)
 		(property "Reference" "#PWR015"
-			(at 41.91 93.98 0)
+			(at 50.8 93.98 0)
 			(effects
 				(font
@@
 		)
 		(property "Value" "GND"
-			(at 41.91 92.71 0)
+			(at 50.8 92.71 0)
 			(effects
 				(font
@@
 		)
 		(property "Footprint" ""
-			(at 41.91 87.63 0)
+			(at 50.8 87.63 0)
 			(effects
 				(font
@@
 		)
 		(property "Datasheet" ""
-			(at 41.91 87.63 0)
+			(at 50.8 87.63 0)
 			(effects
 				(font
@@
 		)
 		(property "Description" "Power symbol creates a global label with name \"GND\" , ground"
-			(at 41.91 87.63 0)
+			(at 50.8 87.63 0)
 			(effects
 				(font
@@
 	)
 	(symbol
+		(lib_id "power:GNDD")
+		(at 59.69 87.63 0)
+		(unit 1)
+		(exclude_from_sim no)
+		(in_bom yes)
+		(on_board yes)
+		(dnp no)
+		(fields_autoplaced yes)
+		(property "Reference" "#PWR0109"
+			(at 59.69 93.98 0)
+			(effects
+				(font
+					(size 1.27 1.27)
+				)
+				(hide yes)
+			)
+		)
+		(property "Value" "GNDD"
+			(at 59.69 91.44 0)
+			(effects
+				(font
+					(size 1.27 1.27)
+				)
+			)
+		)
+		(property "Footprint" ""
+			(at 59.69 87.63 0)
+			(effects
+				(font
+					(size 1.27 1.27)
+				)
+				(hide yes)
+			)
+		)
+		(property "Datasheet" ""
+			(at 59.69 87.63 0)
+			(effects
+				(font
+					(size 1.27 1.27)
+				)
+				(hide yes)
+			)
+		)
+		(property "Description" "Power symbol creates a global label with name \"GNDD\" , digital ground"
+			(at 59.69 87.63 0)
+			(effects
+				(font
+					(size 1.27 1.27)
+				)
+				(hide yes)
+			)
+		)
+		(pin "1"
+		)
+		(instances
+			(project "463 term project"
+				(path "/9eb85bbe-b7ed-4e10-9c6c-ee118bb46686"
+					(reference "#PWR0109")
+					(unit 1)
+				)
+			)
+		)
+	)
+	(symbol
 		(lib_id "Transistor_BJT:BC547")
 		(at 161.29 189.23 0)
@@
 	)
 	(symbol
+		(lib_id "Device:R")
+		(at 45.72 83.82 90)
+		(unit 1)
+		(exclude_from_sim no)
+		(in_bom yes)
+		(on_board yes)
+		(dnp no)
+		(fields_autoplaced yes)
+		(property "Reference" "R18"
+			(at 45.72 77.47 90)
+			(effects
+				(font
+					(size 1.27 1.27)
+				)
+			)
+		)
+		(property "Value" "0"
+			(at 45.72 80.01 90)
+			(effects
+				(font
+					(size 1.27 1.27)
+				)
+			)
+		)
+		(property "Footprint" "Resistor_THT:R_Axial_DIN0207_L6.3mm_D2.5mm_P10.16mm_Horizontal"
+			(at 45.72 85.598 90)
+			(effects
+				(font
+					(size 1.27 1.27)
+				)
+				(hide yes)
+			)
+		)
+		(property "Datasheet" "~"
+			(at 45.72 83.82 0)
+			(effects
+				(font
+					(size 1.27 1.27)
+				)
+				(hide yes)
+			)
+		)
+		(property "Description" "Resistor"
+			(at 45.72 83.82 0)
+			(effects
+				(font
+					(size 1.27 1.27)
+				)
+				(hide yes)
+			)
+		)
+		(pin "1"
+		)
+		(pin "2"
+		)
+		(instances
+			(project "463 term project"
+				(path "/9eb85bbe-b7ed-4e10-9c6c-ee118bb46686"
+					(reference "R18")
+					(unit 1)
+				)
+			)
+		)
+	)
+	(symbol
 		(lib_id "Diode:1N4001")
 		(at 455.93 220.98 180)
@@
 	)
 	(symbol
+		(lib_id "Device:R")
+		(at 55.88 83.82 90)
+		(unit 1)
+		(exclude_from_sim no)
+		(in_bom yes)
+		(on_board yes)
+		(dnp no)
+		(fields_autoplaced yes)
+		(property "Reference" "R19"
+			(at 55.88 77.47 90)
+			(effects
+				(font
+					(size 1.27 1.27)
+				)
+			)
+		)
+		(property "Value" "0"
+			(at 55.88 80.01 90)
+			(effects
+				(font
+					(size 1.27 1.27)
+				)
+			)
+		)
+		(property "Footprint" "Resistor_THT:R_Axial_DIN0207_L6.3mm_D2.5mm_P10.16mm_Horizontal"
+			(at 55.88 85.598 90)
+			(effects
+				(font
+					(size 1.27 1.27)
+				)
+				(hide yes)
+			)
+		)
+		(property "Datasheet" "~"
+			(at 55.88 83.82 0)
+			(effects
+				(font
+					(size 1.27 1.27)
+				)
+				(hide yes)
+			)
+		)
+		(property "Description" "Resistor"
+			(at 55.88 83.82 0)
+			(effects
+				(font
+					(size 1.27 1.27)
+				)
+				(hide yes)
+			)
+		)
+		(pin "1"
+		)
+		(pin "2"
+		)
+		(instances
+			(project "463 term project"
+				(path "/9eb85bbe-b7ed-4e10-9c6c-ee118bb46686"
+					(reference "R19")
+					(unit 1)
+				)
+			)
+		)
+	)
+	(symbol
 		(lib_id "Connector:Conn_01x02_Pin")
 		(at 271.78 262.89 0)
@@
 	(symbol
 		(lib_id "power:GNDPWR")
-		(at 50.8 87.63 0)
+		(at 41.91 87.63 0)
+		(mirror y)
 		(unit 1)
 		(exclude_from_sim no)
@@
 		(fields_autoplaced yes)
 		(property "Reference" "#PWR094"
-			(at 50.8 92.71 0)
+			(at 41.91 92.71 0)
 			(effects
 				(font
@@
 		)
 		(property "Value" "GNDPWR"
-			(at 50.673 91.44 0)
+			(at 42.037 91.44 0)
 			(effects
 				(font
@@
 		)
 		(property "Footprint" ""
-			(at 50.8 88.9 0)
+			(at 41.91 88.9 0)
 			(effects
 				(font
@@
 		)
 		(property "Datasheet" ""
-			(at 50.8 88.9 0)
+			(at 41.91 88.9 0)
 			(effects
 				(font
@@
 		)
 		(property "Description" "Power symbol creates a global label with name \"GNDPWR\" , global ground"
-			(at 50.8 87.63 0)
+			(at 41.91 87.63 0)
 			(effects
 				(font

Commit message: Updates on Layout and Schematic
Parts:
- removed R19: 0, Resistor_THT:R_Axial_DIN0207_L6.3mm_D2.5mm_P10.16mm_Horizontal, symbol Device:R
Changed lines of the file:
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@@
 	)
 	(junction
-		(at 50.8 83.82)
-		(diameter 0)
-		(color 0 0 0 0)
-	)
-	(junction
 		(at 167.64 267.97)
 		(diameter 0)
@@
 	(wire
 		(pts
-			(xy 59.69 83.82) (xy 59.69 87.63)
-		)
-		(stroke
-			(width 0)
-			(type default)
-		)
-	)
-	(wire
-		(pts
 			(xy 226.06 148.59) (xy 223.52 148.59)
 		)
@@
 	(wire
 		(pts
-			(xy 50.8 83.82) (xy 52.07 83.82)
-		)
-		(stroke
-			(width 0)
-			(type default)
-		)
-	)
-	(wire
-		(pts
 			(xy 139.7 175.26) (xy 163.83 175.26)
 		)
@@
 	)
 	(symbol
-		(lib_id "power:GNDD")
-		(at 59.69 87.63 0)
-		(unit 1)
-		(exclude_from_sim no)
-		(in_bom yes)
-		(on_board yes)
-		(dnp no)
-		(fields_autoplaced yes)
-		(property "Reference" "#PWR0109"
-			(at 59.69 93.98 0)
-			(effects
-				(font
-					(size 1.27 1.27)
-				)
-				(hide yes)
-			)
-		)
-		(property "Value" "GNDD"
-			(at 59.69 91.44 0)
-			(effects
-				(font
-					(size 1.27 1.27)
-				)
-			)
-		)
-		(property "Footprint" ""
-			(at 59.69 87.63 0)
-			(effects
-				(font
-					(size 1.27 1.27)
-				)
-				(hide yes)
-			)
-		)
-		(property "Datasheet" ""
-			(at 59.69 87.63 0)
-			(effects
-				(font
-					(size 1.27 1.27)
-				)
-				(hide yes)
-			)
-		)
-		(property "Description" "Power symbol creates a global label with name \"GNDD\" , digital ground"
-			(at 59.69 87.63 0)
-			(effects
-				(font
-					(size 1.27 1.27)
-				)
-				(hide yes)
-			)
-		)
-		(pin "1"
-		)
-		(instances
-			(project "463 term project"
-				(path "/9eb85bbe-b7ed-4e10-9c6c-ee118bb46686"
-					(reference "#PWR0109")
-					(unit 1)
-				)
-			)
-		)
-	)
-	(symbol
 		(lib_id "Transistor_BJT:BC547")
 		(at 161.29 189.23 0)
@@
 					(unit 1)
 				)
-			)
-		)
-	)
-	(symbol
-		(lib_id "Device:R")
-		(at 55.88 83.82 90)
-		(unit 1)
-		(exclude_from_sim no)
-		(in_bom yes)
-		(on_board yes)
-		(dnp no)
-		(fields_autoplaced yes)
-		(property "Reference" "R19"
-			(at 55.88 77.47 90)
-			(effects
-				(font
-					(size 1.27 1.27)
-				)
-			)
-		)
-		(property "Value" "0"
-			(at 55.88 80.01 90)
-			(effects
-				(font
-					(size 1.27 1.27)
-				)
-			)
-		)
-		(property "Footprint" "Resistor_THT:R_Axial_DIN0207_L6.3mm_D2.5mm_P10.16mm_Horizontal"
-			(at 55.88 85.598 90)
-			(effects
-				(font
-					(size 1.27 1.27)
-				)
-				(hide yes)
-			)
-		)
-		(property "Datasheet" "~"
-			(at 55.88 83.82 0)
-			(effects
-				(font
-					(size 1.27 1.27)
-				)
-				(hide yes)
-			)
-		)
-		(property "Description" "Resistor"
-			(at 55.88 83.82 0)
-			(effects
-				(font
-					(size 1.27 1.27)
-				)
-				(hide yes)
-			)
-		)
-		(pin "1"
-		)
-		(pin "2"
-		)
-		(instances
-			(project "463 term project"
-				(path "/9eb85bbe-b7ed-4e10-9c6c-ee118bb46686"
-					(reference "R19")
-					(unit 1)
-				)
