File: [02]Designs/KiCad Designs/463 term project.kicad_sch (KiCad schematic)
At the start: 143 parts, among them J1 Conn_01x02_Pin, J10 Conn_01x01_Pin, J11 Conn_01x01_Pin, J12 Conn_01x01_Pin, J13 Conn_01x01_Pin, J14 Conn_01x01_Pin, J15 Conn_01x01_Pin, J16 Conn_01x01_Pin, J17 Conn_01x01_Pin, J18 Conn_01x02_Pin, J19 Conn_01x02_Pin, J2 Screw_Terminal_01x01, J20 Conn_01x02_Pin, J21 Conn_01x02_Pin, J22 Conn_01x02_Pin, J23 Conn_01x02_Pin, J24 Conn_01x02_Pin, J25 Conn_01x02_Pin, J26 Conn_01x02_Pin, J3 Screw_Terminal_01x01, J4 Conn_01x03_Pin, J5 Screw_Terminal_01x01, J6 Screw_Terminal_01x01, J7 Conn_01x02_Pin, J8 Conn_01x01_Pin, J9 Conn_01x01_Pin, Q1 BC547, Q10 PJMH099N60EC, Q11 PJMH099N60EC, Q2 BC547, Q7 PJMH099N60EC, Q8 PJMH099N60EC, Q9 PJMH099N60EC, SW1 SW_Nidec_CAS-120A1, T2 Transformer, U1 6N135, U10 ADuM1200AR, U11 IR2110, U12 LM7805_TO220, U14 LM7815_TO220, U16 LD1117S33TR_SOT223, U17 LD1117S33TR_SOT223, U18 5 Button Module, U19 LM7812_TO220, U2 6N135, U20 LM7812_TO220, U3 74HC00, U4 IR2110, U5 IR2110, U6 ACS712xLCTR-30A, U8 ADuM1200AR, U9 ADuM1200AR

Commit message: Reduced PCB Size
This reverts commit fabae2b9b95dacba0e962aa67e5fb78db473a071.
Connections:
- net 220V_Line: now also T2.10 (AB); no longer T2.6 (AA)
- net 220V_Neutral: now also T2.6 (AA); no longer T2.10 (AB)
- net at D5.2 (A): now also T2.1 (SD); no longer T2.5 (SA)
- net at D24.2 (A): now also T2.5 (SA); no longer T2.1 (SD)
Other:
- moved on the sheet: D24, D5
Changed lines of the file:
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@@
 	(wire
 		(pts
-			(xy 33.02 256.54) (xy 44.45 256.54)
-		)
-		(stroke
-			(width 0)
-			(type default)
-		)
-	)
-	(wire
-		(pts
 			(xy 151.13 113.03) (xy 151.13 116.84)
 		)
@@
 	(wire
 		(pts
+			(xy 30.48 256.54) (xy 44.45 256.54)
+		)
+		(stroke
+			(width 0)
+			(type default)
+		)
+	)
+	(wire
+		(pts
 			(xy 471.17 336.55) (xy 471.17 337.82)
 		)
@@
 		)
 	)
+	(global_label "220V_Line"
+		(shape input)
+		(at 30.48 256.54 180)
+		(fields_autoplaced yes)
+		(effects
+			(font
+				(size 1.27 1.27)
+			)
+			(justify right)
+		)
+		(property "Intersheetrefs" "${INTERSHEET_REFS}"
+			(at 17.9396 256.54 0)
+			(effects
+				(font
+					(size 1.27 1.27)
+				)
+				(justify right)
+				(hide yes)
+			)
+		)
+	)
 	(global_label "+5V_Isolated"
 		(shape input)
@@
 		)
 	)
-	(global_label "220V_Line"
-		(shape input)
-		(at 30.48 246.38 180)
-		(fields_autoplaced yes)
-		(effects
-			(font
-				(size 1.27 1.27)
-			)
-			(justify right)
-		)
-		(property "Intersheetrefs" "${INTERSHEET_REFS}"
-			(at 17.9396 246.38 0)
-			(effects
-				(font
-					(size 1.27 1.27)
-				)
-				(justify right)
-				(hide yes)
-			)
-		)
-	)
 	(global_label "Direction"
 		(shape input)
@@
 		)
 	)
-	(global_label "220V_Neutral"
+	(global_label "Speed_meas"
 		(shape input)
-		(at 33.02 256.54 180)
+		(at 562.61 334.01 0)
 		(fields_autoplaced yes)
 		(effects
@@
 				(size 1.27 1.27)
 			)
-			(justify right)
+			(justify left)
 		)
 		(property "Intersheetrefs" "${INTERSHEET_REFS}"
-			(at 17.4559 256.54 0)
+			(at 577.2065 334.01 0)
 			(effects
 				(font
 					(size 1.27 1.27)
 				)
-				(justify right)
+				(justify left)
 				(hide yes)
 			)
 		)
 	)
-	(global_label "Speed_meas"
+	(global_label "Button1"
 		(shape input)
-		(at 562.61 334.01 0)
+		(at 336.55 280.67 0)
 		(fields_autoplaced yes)
 		(effects
@@
 		)
 		(property "Intersheetrefs" "${INTERSHEET_REFS}"
-			(at 577.2065 334.01 0)
+			(at 346.9131 280.67 0)
 			(effects
 				(font
@@
 		)
 	)
-	(global_label "Button1"
+	(global_label "220V_Neutral"
 		(shape input)
-		(at 336.55 280.67 0)
+		(at 30.48 246.38 180)
 		(fields_autoplaced yes)
 		(effects
@@
 				(size 1.27 1.27)
 			)
-			(justify left)
+			(justify right)
 		)
 		(property "Intersheetrefs" "${INTERSHEET_REFS}"
-			(at 346.9131 280.67 0)
+			(at 14.9159 246.38 0)
 			(effects
 				(font
 					(size 1.27 1.27)
 				)
-				(justify left)
+				(justify right)
 				(hide yes)
 			)
@@
 	(symbol
 		(lib_id "Diode:1N5408")
-		(at 82.55 241.3 180)
+		(at 82.55 261.62 180)
 		(unit 1)
 		(exclude_from_sim no)
@@
 		(fields_autoplaced yes)
 		(property "Reference" "D5"
-			(at 82.55 234.95 0)
+			(at 82.55 255.27 0)
 			(effects
 				(font
@@
 		)
 		(property "Value" "1N5408"
-			(at 82.55 237.49 0)
+			(at 82.55 257.81 0)
 			(effects
 				(font
@@
 		)
 		(property "Footprint" "Diode_THT:D_DO-201AD_P15.24mm_Horizontal"
-			(at 82.55 236.855 0)
+			(at 82.55 257.175 0)
 			(effects
 				(font
@@
 		)
 		(property "Datasheet" "http://www.vishay.com/docs/88516/1n5400.pdf"
-			(at 82.55 241.3 0)
+			(at 82.55 261.62 0)
 			(effects
 				(font
@@
 		)
 		(property "Description" "1000V 3A General Purpose Rectifier Diode, DO-201AD"
-			(at 82.55 241.3 0)
+			(at 82.55 261.62 0)
 			(effects
 				(font
@@
 		)
 		(property "Sim.Device" "D"
-			(at 82.55 241.3 0)
+			(at 82.55 261.62 0)
 			(effects
 				(font
@@
 		)
 		(property "Sim.Pins" "1=K 2=A"
-			(at 82.55 241.3 0)
+			(at 82.55 261.62 0)
 			(effects
 				(font
@@
 		)
 		(instances
-			(project ""
+			(project "463 term project"
 				(path "/9eb85bbe-b7ed-4e10-9c6c-ee118bb46686"
 					(reference "D5")
@@
 	(symbol
 		(lib_id "Diode:1N5408")
-		(at 82.55 261.62 180)
+		(at 82.55 241.3 180)
 		(unit 1)
 		(exclude_from_sim no)
@@
 		(on_board yes)
 		(dnp no)
-		(fields_autoplaced yes)
 		(property "Reference" "D24"
-			(at 82.55 255.27 0)
+			(at 82.55 234.95 0)
 			(effects
 				(font
@@
 		)
 		(property "Value" "1N5408"
-			(at 82.55 257.81 0)
+			(at 82.55 237.49 0)
 			(effects
 				(font
@@
 		)
 		(property "Footprint" "Diode_THT:D_DO-201AD_P15.24mm_Horizontal"
-			(at 82.55 257.175 0)
+			(at 82.55 236.855 0)
 			(effects
 				(font
@@
 		)
 		(property "Datasheet" "http://www.vishay.com/docs/88516/1n5400.pdf"
-			(at 82.55 261.62 0)
+			(at 82.55 241.3 0)
 			(effects
 				(font
@@
 		)
 		(property "Description" "1000V 3A General Purpose Rectifier Diode, DO-201AD"
-			(at 82.55 261.62 0)
+			(at 82.55 241.3 0)
 			(effects
 				(font
@@
 		)
 		(property "Sim.Device" "D"
-			(at 82.55 261.62 0)
+			(at 82.55 241.3 0)
 			(effects
 				(font
@@
 		)
 		(property "Sim.Pins" "1=K 2=A"
-			(at 82.55 261.62 0)
+			(at 82.55 241.3 0)
 			(effects
 				(font
