File: [02]Designs/KiCad Designs/463 term project.kicad_pcb (KiCad board)
At the start: 2 copper layers, 114 parts, among them J2 Screw_Terminal_01x01, J3 Screw_Terminal_01x01, Q1 BC547, Q10 PJMH099N60EC, Q11 PJMH099N60EC, Q2 BC547, Q7 PJMH099N60EC, Q8 PJMH099N60EC, Q9 PJMH099N60EC, T1 Transformer_1P_2S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

Commit message: Layout.v1 finished & Schematic updates
Co-Authored-By: KaanDemirkoparan <57269134+KaanDemirkoparan@users.noreply.github.com>
Parts:
- removed C5: 100n, Capacitor_THT:C_Disc_D5.0mm_W2.5mm_P5.00mm
- removed D1, D2: D, Diode_THT:D_DO-35_SOD27_P10.16mm_Horizontal
- removed T1: Transformer_1P_2S, Transformer_THT:Transformer_Breve_TEZ-35x42
- removed U13: LM7812_TO220, Package_TO_SOT_THT:TO-220-3_Vertical
- removed U15: LM78L05_SO8, Package_SO:SOIC-8_3.9x4.9mm_P1.27mm
- added C43: 100n, Capacitor_THT:C_Disc_D5.0mm_W2.5mm_P5.00mm, F.Cu at (285.2, 144.6)
- added D10: LED, METUPowerLab_LEDs_SurfaceMounts:0603 Medium, F.Cu at (260.4, 180.6)
- added D21: LED, METUPowerLab_LEDs_SurfaceMounts:0603 Medium, F.Cu at (262.9, 180.5)
- added D22: LED, METUPowerLab_LEDs_SurfaceMounts:0603 Medium, F.Cu at (265.3, 180.6)
- added D23: LED, METUPowerLab_LEDs_SurfaceMounts:0603 Medium, F.Cu at (267.6, 180.6)
- added D24: 1N5408, Diode_THT:D_DO-201AD_P15.24mm_Horizontal, F.Cu at (118.8, 132.9)
- added D5: 1N5408, Diode_THT:D_DO-201AD_P15.24mm_Horizontal, F.Cu at (118.8, 112.9)
- added J5: Screw_Terminal_01x01, METUPowerLab_Boards_ESP32:Untitled, F.Cu at (220.6, 82.5)
- added J6: Screw_Terminal_01x01, METUPowerLab_Boards_ESP32:Untitled, F.Cu at (204.3, 82.7)
- added R16: 1k, Resistor_THT:R_Axial_DIN0207_L6.3mm_D2.5mm_P10.16mm_Horizontal, F.Cu at (290.1, 121.1)
- added R17: 1k, Resistor_THT:R_Axial_DIN0207_L6.3mm_D2.5mm_P10.16mm_Horizontal, F.Cu at (290.1, 144.7)
- added R29: 10K, METUPowerLab_Resistors_ChipResistors:0603 Medium, F.Cu at (260.0, 177.3)
- added R30: 10K, METUPowerLab_Resistors_ChipResistors:0603 Medium, F.Cu at (262.7, 177.1)
- added R31: 10K, METUPowerLab_Resistors_ChipResistors:0603 Medium, F.Cu at (265.4, 177.2)
- added R32: 10K, METUPowerLab_Resistors_ChipResistors:0603 Medium, F.Cu at (267.9, 177.2)
- added RV1: R_Potentiometer, Connector_PinHeader_2.54mm:PinHeader_1x03_P2.54mm_Vertical, F.Cu at (295.4, 131.4)
- added SW1: SW_Nidec_CAS-120A1, Connector_PinHeader_2.54mm:PinHeader_1x03_P2.54mm_Vertical, F.Cu at (295.4, 121.7)
- added T2: Transformer, Transformer_THT:Transformer_Breve_TEZ-35x42, F.Cu at (90.5, 132.9)
- added U19: LM7812_TO220, Package_TO_SOT_THT:TO-220-3_Vertical, F.Cu at (136.6, 125.0)
- added U20: LM7812_TO220, Package_TO_SOT_THT:TO-220-3_Vertical, F.Cu at (136.9, 107.5)
- U12: value LM7812_TO220 -> LM7805_TO220
- U16, U17: footprint Package_TO_SOT_SMD:SOT-223-3_TabPin2 -> Package_TO_SOT_THT:TO-220-3_Vertical
- moved R14 207.2 mm to (280.9, 96.7), turned to 180 degrees
- moved R15 191.5 mm to (259.9, 84.5)
- moved D19 178.9 mm to (271.0, 102.2)
- moved R6 176.0 mm to (250.0, 69.2), turned to 90 degrees
- moved D20 173.4 mm to (264.5, 98.3), turned to 90 degrees
- moved R8 173.2 mm to (243.8, 66.0), turned to 180 degrees
- moved U7 171.1 mm to (239.4, 148.5), turned to -90 degrees
- moved D14 165.1 mm to (255.7, 69.3), turned to 90 degrees
- moved R5 165.1 mm to (244.1, 108.1), turned to 180 degrees
- moved C25 163.0 mm to (290.6, 108.2)
- moved R1 162.3 mm to (217.3, 175.9), turned to 180 degrees
- moved C1 162.1 mm to (227.1, 175.7)
- moved R2 160.6 mm to (215.2, 179.9), turned to 180 degrees
- moved J2 150.2 mm to (274.3, 63.9)
- moved J3 146.7 mm to (274.3, 79.9)
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Connections:
- C29 pad 1: Net-(D1-K) -> Net-(D24-K)
- C30 pad 1: Net-(D1-K) -> Net-(D24-K)
- C31 pad 1: Net-(D1-K) -> Net-(D24-K)
- C32 pad 1: Net-(D1-K) -> Net-(D24-K)
- C33 pad 1: Net-(U12-VO) -> Net-(U12-VI)
- C36 pad 1: Net-(U12-VO) -> Net-(U12-VI)
- U12 pad 1: Net-(D1-K) -> Net-(U12-VI)
- U12 pad 3: Net-(U12-VO) -> +5V
- U14 pad 1: Net-(D1-K) -> Net-(D24-K)
- U7 pad 12: unconnected-(U7-IO14-Pad12) -> POT
- U7 pad 13: /LED -> unconnected-(U7-IO12-Pad13)
- U7 pad 26: unconnected-(U7-IO4-Pad26) -> /LED_cw
- U7 pad 29: unconnected-(U7-IO5-Pad29) -> /LED_ccw
- U7 pad 33: unconnected-(U7-IO21-Pad33) -> /LED_debug
- U7 pad 36: unconnected-(U7-IO22-Pad36) -> /LED_brake
- U7 pad 37: unconnected-(U7-IO23-Pad37) -> /LED
- U7 pad 5: unconnected-(U7-IO34-Pad5) -> Direction

Commit message: Layout and schematic updates
Co-Authored-By: KaanDemirkoparan <57269134+KaanDemirkoparan@users.noreply.github.com>
Parts:
- removed JP6, JP7, JP8, JP9: SolderJumper_2_Open, Jumper:SolderJumper-2_P1.3mm_Open_TrianglePad1.0x1.5mm
- added J1: Conn_01x02_Pin, Connector_PinHeader_2.54mm:PinHeader_1x02_P2.54mm_Vertical, F.Cu at (131.2, 162.0)
- added J10: Conn_01x01_Pin, Connector_Wire:SolderWirePad_1x01_SMD_5x10mm, F.Cu at (223.0, 76.1)
- added J11: Conn_01x01_Pin, Connector_Wire:SolderWirePad_1x01_SMD_5x10mm, F.Cu at (206.7, 76.6)
- added J12: Conn_01x01_Pin, Connector_Wire:SolderWirePad_1x01_SMD_5x10mm, F.Cu at (287.7, 61.3)
- added J13: Conn_01x01_Pin, Connector_Wire:SolderWirePad_1x01_SMD_5x10mm, F.Cu at (287.7, 77.3)
- added J14: Conn_01x01_Pin, Connector_Wire:SolderWirePad_1x01_SMD_1x2mm, F.Cu at (101.0, 157.3)
- added J15: Conn_01x01_Pin, Connector_Wire:SolderWirePad_1x01_SMD_1x2mm, F.Cu at (101.0, 163.0)
- added J16: Conn_01x01_Pin, Connector_Wire:SolderWirePad_1x01_SMD_5x10mm, F.Cu at (57.3, 177.0)
- added J17: Conn_01x01_Pin, Connector_Wire:SolderWirePad_1x01_SMD_5x10mm, F.Cu at (56.9, 163.2)
- added J18: Conn_01x02_Pin, Connector_PinHeader_2.54mm:PinHeader_1x02_P2.54mm_Vertical, F.Cu at (212.7, 135.5)
- added J19: Conn_01x02_Pin, Connector_PinHeader_2.54mm:PinHeader_1x02_P2.54mm_Vertical, F.Cu at (203.4, 148.3)
- added J20: Conn_01x02_Pin, Connector_PinHeader_2.54mm:PinHeader_1x02_P2.54mm_Vertical, F.Cu at (210.1, 148.3)
- added J7: Conn_01x02_Pin, Connector_PinHeader_2.54mm:PinHeader_1x02_P2.54mm_Vertical, F.Cu at (204.8, 135.5)
- added J8: Conn_01x01_Pin, Connector_Wire:SolderWirePad_1x01_SMD_5x10mm, F.Cu at (60.6, 80.7)
- added J9: Conn_01x01_Pin, Connector_Wire:SolderWirePad_1x01_SMD_5x10mm, F.Cu at (58.7, 62.7)
- moved D6 162.7 mm to (270.5, 180.6), turned to -90 degrees
- moved R28 161.2 mm to (270.5, 177.2), turned to -90 degrees
- moved C41 35.7 mm to (112.5, 159.4)
- moved C42 35.7 mm to (121.6, 159.4)
- moved U17 35.7 mm to (107.7, 162.9)
- moved U3 13.9 mm to (204.6, 158.1), turned to 0 degrees
- moved C20 11.3 mm to (161.1, 63.4)
- moved C21 6.34 mm to (161.1, 60.4)
- moved R1 5.41 mm to (217.5, 181.3)
- moved R2 3.57 mm to (217.5, 177.2)
- moved D9 0.87 mm to (66.0, 86.7)
Connections:
- net Net-(D11-K) renamed /S4_Drain
- net Net-(D7-K) renamed Current_Sense_out
- net Q7_Drain renamed S3_Drain
- C41 pad 1: +3.3V_Isolated -> Net-(J1-Pin_2)
- C42 pad 1: +3.3V_Isolated -> Net-(J1-Pin_2)
- JP11 pad 2: S1_ISO -> S2_ISO
- JP13 pad 2: S3_ISO -> S4_ISO
- U17 pad 2: +3.3V_Isolated -> Net-(J1-Pin_2)
Routing:
- net +3.3V_Isolated: track 0.00 -> 446.7 mm
- net I_meas: track 0.00 -> 262.8 mm
- net +5V: track 0.00 -> 218.2 mm
- net +12V: track 0.00 -> 214.2 mm
- net 220V_Neutral: track 0.00 -> 142.7 mm
- net 220V_Line: track 0.00 -> 129.9 mm
- net Net-(D24-K): track 0.00 -> 97.7 mm
- net Net-(D14-K): track 0.00 -> 88.9 mm
- net Net-(D16-K): track 0.00 -> 64.6 mm
- net S3: track 0.00 -> 63.9 mm
- net Net-(R1-Pad2): track 0.00 -> 53.5 mm
- net S1: track 0.00 -> 49.5 mm
- net Net-(R2-Pad2): track 0.00 -> 39.1 mm
- net Net-(D15-K): track 0.00 -> 34.5 mm
- net DC_200V: track 0.00 -> 33.9 mm
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- added copper zone on F.Cu, net /S4_Drain
- added copper zone on F.Cu, net Current_Sense_out
- added copper zone on F.Cu, net DC_200V
- added copper zone on F.Cu, net Q11_Drain
- added copper zone on F.Cu, net S3_Drain

Commit message: [Design] Layout Finished
Parts:
- removed JP10, JP11, JP12, JP13, JP14, JP15: SolderJumper_2_Open, Jumper:SolderJumper-2_P1.3mm_Open_TrianglePad1.0x1.5mm
- added J21: Conn_01x02_Pin, Connector_PinHeader_2.54mm:PinHeader_1x02_P2.54mm_Vertical, F.Cu at (232.0, 142.5)
- added J22: Conn_01x02_Pin, Connector_PinHeader_2.54mm:PinHeader_1x02_P2.54mm_Vertical, F.Cu at (276.6, 143.5)
- added J23: Conn_01x02_Pin, Connector_PinHeader_2.54mm:PinHeader_1x02_P2.54mm_Vertical, F.Cu at (271.9, 143.5)
- added J24: Conn_01x02_Pin, Connector_PinHeader_2.54mm:PinHeader_1x02_P2.54mm_Vertical, F.Cu at (267.3, 143.5)
- added J25: Conn_01x02_Pin, Connector_PinHeader_2.54mm:PinHeader_1x02_P2.54mm_Vertical, F.Cu at (262.6, 143.5)
- added J26: Conn_01x02_Pin, Connector_PinHeader_2.54mm:PinHeader_1x02_P2.54mm_Vertical, F.Cu at (258.0, 143.5)
- added J4: Conn_01x03_Pin, Connector_PinHeader_2.54mm:PinHeader_1x03_P2.54mm_Vertical, F.Cu at (292.8, 136.0)
- D9: moved to B.Cu
- U18: value ~ -> 5 Button Module
- moved R1 20.0 mm to (198.5, 175.2), turned to 90 degrees
- moved R12 14.4 mm to (181.5, 87.4), turned to -90 degrees
- moved D6 13.9 mm to (284.4, 179.7), turned to 90 degrees
- moved R28 12.0 mm to (282.6, 177.2), turned to 0 degrees
- moved D23 10.3 mm to (277.9, 179.7), turned to 90 degrees
- moved R32 8.16 mm to (276.1, 177.2), turned to 0 degrees
- moved J17 7.89 mm to (54.5, 155.8), turned to 180 degrees
- moved D22 5.88 mm to (271.1, 179.7), turned to 90 degrees
- moved R29 5.50 mm to (254.6, 177.2), turned to 0 degrees
- moved C43 5.27 mm to (285.5, 139.3)
- moved R16 5.25 mm to (289.1, 115.9)
- moved R17 5.25 mm to (289.1, 139.5)
- moved RV1 5.03 mm to (292.9, 127.0)
- moved SW1 5.03 mm to (292.9, 117.4)
- moved D17 4.83 mm to (176.0, 106.8)
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Connections:
- C10 pad 2: GND -> GNDPWR
- C11 pad 2: GND -> GNDPWR
- C14 pad 2: GND -> GNDPWR
- C15 pad 2: GND -> GNDPWR
- C18 pad 2: GND -> GNDPWR
- C19 pad 2: GND -> GNDPWR
- C22 pad 1: GND -> GNDPWR
- C24 pad 2: GND -> GNDPWR
- C25 pad 2: GND -> GNDPWR
- D11 pad 2: GND -> GNDPWR
- D12 pad 2: GND -> GNDPWR
- D9 pad 2: 220V_Line -> 220V_Neutral
- D9 pad 3: GND -> GNDPWR
- D9 pad 4: 220V_Neutral -> 220V_Line
- Q10 pad 3: GND -> GNDPWR
- Q11 pad 3: GND -> GNDPWR
- Q7 pad 3: GND -> GNDPWR
- R12 pad 1: GND -> GNDPWR
- R13 pad 2: GND -> GNDPWR
- R15 pad 1: GND -> GNDPWR
- R7 pad 1: GND -> GNDPWR
- U11 pad 2: GND -> GNDPWR
- U4 pad 2: GND -> GNDPWR
- U5 pad 2: GND -> GNDPWR
Routing:
- net +5V_Isolated: track 9.26 -> 323.5 mm, vias 0 -> 1
- net DGND_Isolated: track 9.14 -> 251.1 mm, vias 1 -> 4
- net Button1: track 0.00 -> 130.5 mm
- net Button2: track 0.00 -> 127.5 mm
- net Button3: track 0.00 -> 116.3 mm
- net Button4: track 0.00 -> 108.1 mm
- net Button5: track 0.00 -> 97.3 mm
- net S4_ISO: track 0.00 -> 85.0 mm
- net S2_ISO: track 0.00 -> 82.7 mm
- net Direction: track 0.00 -> 56.8 mm
- net POT: track 0.00 -> 47.3 mm
- net +5V: track 218.2 -> 261.2 mm
- net S3_ISO: track 0.00 -> 38.2 mm
- net +3.3V_Isolated: track 446.7 -> 484.4 mm
- net H_IN: track 0.00 -> 36.8 mm
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- added copper zone on B.Cu, net DGND_Isolated
- added copper zone on B.Cu, net GND
- added copper zone on F.Cu, net GND
- added copper zone on B.Cu, net GNDPWR
Other:
- board outline added: 250 x 135 mm

Commit message: [Design] Layout Finalized
Parts:
- added R18: 0, Resistor_THT:R_Axial_DIN0207_L6.3mm_D2.5mm_P10.16mm_Horizontal, F.Cu at (113.5, 93.2)
- added R19: 0, Resistor_THT:R_Axial_DIN0207_L6.3mm_D2.5mm_P10.16mm_Horizontal, F.Cu at (129.2, 144.4)
- moved U17 37.9 mm to (145.6, 163.0)
- moved C41 37.9 mm to (150.4, 159.5)
- moved C42 37.9 mm to (159.5, 159.4)
- moved J14 37.9 mm to (138.9, 157.3)
- moved J15 37.9 mm to (138.9, 163.1)
- moved J1 37.9 mm to (169.1, 162.1)
- moved R12 10.7 mm to (171.2, 90.2), turned to 0 degrees
- moved D12 8.34 mm to (238.7, 102.4)
- moved Q10 7.94 mm to (181.3, 94.8)
- moved D11 7.45 mm to (187.2, 102.4)
- moved Q7 6.80 mm to (232.8, 94.8)
- moved R7 4.75 mm to (218.7, 94.0)
- moved J6 2.80 mm to (207.0, 82.0)
- moved J5 1.69 mm to (219.0, 82.0)
- moved Q9 1.13 mm to (181.3, 60.7)
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Routing:
- net +3.3V_Isolated: track 484.4 -> 433.0 mm
- net DGND_Isolated: track 251.1 -> 289.0 mm
- net +5V_Isolated: track 323.5 -> 285.6 mm
- net Net-(D17-A): track 20.5 -> 27.5 mm
- net Net-(D15-A): track 21.3 -> 25.3 mm
- net S1_ISO: track 34.8 -> 37.7 mm
- net S2_ISO: track 82.7 -> 85.3 mm
- net Net-(D16-K): track 63.7 -> 65.8 mm
- net Net-(D14-K): track 84.2 -> 85.5 mm
- net S3_ISO: track 38.2 -> 38.8 mm
- net Net-(D16-A): track 16.6 -> 16.0 mm
- net /S4_Drain: track 32.4 -> 33.0 mm

Commit message: Updates on Layout and Schematic
Parts:
- removed R19: 0, Resistor_THT:R_Axial_DIN0207_L6.3mm_D2.5mm_P10.16mm_Horizontal

Commit message: Updates on Layout
Routing:
- net 220V_Neutral: track 142.1 -> 138.9 mm
- net Button1: track 130.5 -> 129.0 mm
- net Button4: track 108.1 -> 107.3 mm
- net Button2: track 127.5 -> 126.7 mm
- net Button3: track 116.3 -> 115.6 mm
Other:
- board size 250 x 135 mm -> 250 x 135.5 mm
Changed lines of the file:
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@@
 	(gr_rect
 		(start 50 48)
-		(end 300 183)
+		(end 300 183.5)
 		(stroke
 			(width 0.2)
@@
 	)
 	(segment
-		(start 63.75 80.75)
-		(end 60.66 80.75)
-		(width 6)
-		(layer "F.Cu")
-		(net 20)
-	)
-	(segment
-		(start 60.66 80.75)
-		(end 60.57 80.66)
-		(width 6)
-		(layer "F.Cu")
-		(net 20)
-	)
-	(segment
 		(start 72.75 92.67)
 		(end 67.19 92.67)
@@
 	)
 	(segment
-		(start 152.99 181.25)
-		(end 227.75 181.25)
-		(width 0.2)
+		(start 150.42 178.68)
+		(end 152.74 181)
+		(width 0.5)
 		(layer "F.Cu")
 		(net 63)
 	)
 	(segment
-		(start 238.599 170.401)
-		(end 256.231 170.401)
-		(width 0.2)
+		(start 238.75 171)
+		(end 256.83 171)
+		(width 0.5)
 		(layer "F.Cu")
 		(net 63)
 	)
 	(segment
-		(start 227.75 181.25)
-		(end 238.599 170.401)
-		(width 0.2)
+		(start 152.74 181)
+		(end 228.75 181)
+		(width 0.5)
 		(layer "F.Cu")
 		(net 63)
 	)
 	(segment
-		(start 256.231 170.401)
+		(start 256.83 171)
 		(end 259.74 173.91)
-		(width 0.2)
+		(width 0.5)
 		(layer "F.Cu")
 		(net 63)
 	)
 	(segment
-		(start 150.42 178.68)
-		(end 152.99 181.25)
-		(width 0.2)
+		(start 228.75 181)
+		(end 238.75 171)
+		(width 0.5)
 		(layer "F.Cu")
 		(net 63)
@@
 	)
 	(segment
-		(start 126.79 182.25)
-		(end 228.25 182.25)
-		(width 0.2)
+		(start 123.22 178.68)
+		(end 127.04 182.5)
+		(width 0.5)
 		(layer "F.Cu")
 		(net 69)
 	)
 	(segment
-		(start 244.88 171.75)
-		(end 247.04 173.91)
-		(width 0.2)
+		(start 127.04 182.5)
+		(end 238.45 182.5)
+		(width 0.5)
 		(layer "F.Cu")
 		(net 69)
 	)
 	(segment
-		(start 238.75 171.75)
-		(end 244.88 171.75)
-		(width 0.2)
+		(start 238.45 182.5)
+		(end 247.04 173.91)
+		(width 0.5)
 		(layer "F.Cu")
 		(net 69)
 	)
 	(segment
-		(start 123.22 178.68)
-		(end 126.79 182.25)
-		(width 0.2)
+		(start 185.25 177.75)
+		(end 184 176.5)
+		(width 0.5)
 		(layer "F.Cu")
-		(net 69)
+		(net 70)
 	)
 	(segment
-		(start 228.25 182.25)
-		(end 238.75 171.75)
-		(width 0.2)
+		(start 177.62 177.13)
+		(end 177.62 178.68)
+		(width 0.5)
 		(layer "F.Cu")
-		(net 69)
+		(net 70)
 	)
 	(segment
-		(start 179.19 180.25)
-		(end 227.25 180.25)
-		(width 0.2)
+		(start 184 176.5)
+		(end 178.25 176.5)
+		(width 0.5)
 		(layer "F.Cu")
 		(net 70)
 	)
 	(segment
-		(start 227.25 180.25)
-		(end 238.75 168.75)
-		(width 0.2)
+		(start 267.36 173.91)
+		(end 262.45 169)
+		(width 0.5)
 		(layer "F.Cu")
 		(net 70)
 	)
 	(segment
-		(start 262.2 168.75)
-		(end 267.36 173.91)
-		(width 0.2)
+		(start 178.25 176.5)
+		(end 177.62 177.13)
+		(width 0.5)
 		(layer "F.Cu")
 		(net 70)
 	)
 	(segment
-		(start 238.75 168.75)
-		(end 262.2 168.75)
-		(width 0.2)
+		(start 238.25 169)
+		(end 229.5 177.75)
+		(width 0.5)
 		(layer "F.Cu")
 		(net 70)
 	)
 	(segment
-		(start 177.62 178.68)
-		(end 179.19 180.25)
-		(width 0.2)
+		(start 262.45 169)
+		(end 238.25 169)
+		(width 0.5)
+		(layer "F.Cu")
+		(net 70)
+	)
+	(segment
+		(start 229.5 177.75)
+		(end 185.25 177.75)
+		(width 0.5)
 		(layer "F.Cu")
 		(net 70)
@@
 	)
 	(segment
-		(start 227.5 180.75)
-		(end 238.75 169.5)
-		(width 0.2)
+		(start 165.59 180.25)
+		(end 228.25 180.25)
+		(width 0.5)
 		(layer "F.Cu")
 		(net 82)
 	)
 	(segment
-		(start 238.75 169.5)
-		(end 260.41 169.5)
-		(width 0.2)
+		(start 238.5 170)
+		(end 260.91 170)
+		(width 0.5)
 		(layer "F.Cu")
 		(net 82)
 	)
 	(segment
-		(start 166.09 180.75)
-		(end 227.5 180.75)
-		(width 0.2)
+		(start 164.02 178.68)
+		(end 165.59 180.25)
+		(width 0.5)
 		(layer "F.Cu")
 		(net 82)
 	)
 	(segment
-		(start 260.41 169.5)
-		(end 264.82 173.91)
-		(width 0.2)
+		(start 228.25 180.25)
+		(end 238.5 170)
+		(width 0.5)
 		(layer "F.Cu")
 		(net 82)
 	)
 	(segment
-		(start 164.02 178.68)
-		(end 166.09 180.75)
-		(width 0.2)
+		(start 260.91 170)
+		(end 264.82 173.91)
+		(width 0.5)
 		(layer "F.Cu")
 		(net 82)
@@
 	)
 	(segment
-		(start 254.342 171.052)
-		(end 257.2 173.91)
-		(width 0.2)
+		(start 139.89 181.75)
+		(end 229.25 181.75)
+		(width 0.5)
 		(layer "F.Cu")
 		(net 84)
 	)
 	(segment
-		(start 238.698 171.052)
-		(end 254.342 171.052)
-		(width 0.2)
+		(start 255.29 172)
+		(end 257.2 173.91)
+		(width 0.5)
 		(layer "F.Cu")
 		(net 84)
 	)
 	(segment
-		(start 228 181.75)
-		(end 238.698 171.052)
-		(width 0.2)
+		(start 136.82 178.68)
+		(end 139.89 181.75)
+		(width 0.5)
 		(layer "F.Cu")
 		(net 84)
@@
 	)
 	(segment
-		(start 136.82 178.68)
-		(end 139.89 181.75)
-		(width 0.2)
+		(start 239 172)
+		(end 255.29 172)
+		(width 0.5)
 		(layer "F.Cu")
 		(net 84)
 	)
 	(segment
-		(start 139.89 181.75)
-		(end 228 181.75)
+		(start 136.93 178.68)
+		(end 137 178.75)
 		(width 0.2)
 		(layer "F.Cu")
@@
 	)
 	(segment
-		(start 136.93 178.68)
-		(end 137 178.75)
-		(width 0.2)
+		(start 229.25 181.75)
+		(end 239 172)
+		(width 0.5)
 		(layer "F.Cu")
 		(net 84)
@@
 		(polygon
 			(pts
-				(xy 50.5 48.5) (xy 50.5 182.5) (xy 299.5 182.5) (xy 299.5 48.5)
+				(xy 50.5 48.5) (xy 50.5 183) (xy 299.5 183) (xy 299.5 48.5)
 			)
 		)
@@
 		(priority 6)
 		(connect_pads yes
-			(clearance 0.5)
+			(clearance 1)
 		)
 		(min_thickness 0.25)
@@
 				(xy 50.5 150.25) (xy 161.25 150.25) (xy 161.25 156.238103) (xy 170.421065 156.249013) (xy 177.25 149.925926)
 				(xy 177.25 131.5) (xy 187.25 131.5) (xy 187.25 140.5) (xy 196.5 140.5) (xy 196.5 176.25) (xy 237 176.25)
-				(xy 237 139.25) (xy 270 139.25) (xy 270 129.75) (xy 287 129.75) (xy 287 115) (xy 299.5 115) (xy 299.5 182.5)
-				(xy 50.5 182.5)
+				(xy 237 139.25) (xy 270 139.25) (xy 270 129.75) (xy 287 129.75) (xy 287 115) (xy 299.5 115) (xy 299.5 183)
+				(xy 50.5 183)
 			)
 		)

Commit message: Reduced PCB Size
This reverts commit fabae2b9b95dacba0e962aa67e5fb78db473a071.
Parts:
- J16, J17: moved to B.Cu
- moved J12 114.0 mm to (183.8, 14.5)
- moved C17 96.8 mm to (88.8, 86.3)
- moved C37 96.4 mm to (65.3, 87.2)
- moved U16 96.4 mm to (55.5, 90.5)
- moved C39 96.4 mm to (58.9, 94.6)
- moved U12 96.3 mm to (55.5, 81.8)
- moved U19 96.2 mm to (55.5, 73.2)
- moved U14 96.2 mm to (55.6, 64.7)
- moved U20 96.2 mm to (55.9, 55.7)
- moved D20 94.2 mm to (183.5, 50.3)
- moved J13 94.2 mm to (206.7, 29.3)
- moved J22 94.2 mm to (195.6, 95.5)
- moved C16 94.2 mm to (101.9, 85.8)
- moved C18 94.2 mm to (107.6, 32.4)
- moved C2 94.2 mm to (140.3, 110.5)
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Connections:
- T2 pad 1: Net-(D24-A) -> Net-(D5-A)
- T2 pad 10: 220V_Neutral -> 220V_Line
- T2 pad 5: Net-(D5-A) -> Net-(D24-A)
- T2 pad 6: 220V_Line -> 220V_Neutral
Routing:
- net Net-(D5-A): track 13.1 -> 68.3 mm
- net 220V_Neutral: track 138.9 -> 85.4 mm
- net Net-(D24-K): track 97.7 -> 67.4 mm
- net +3.3V_Isolated: track 433.0 -> 407.8 mm
- net Button5: track 97.7 -> 86.2 mm
- net DGND_Isolated: track 289.0 -> 277.6 mm, vias 4 -> 5
- net Button4: track 107.3 -> 96.0 mm
- net Button2: track 126.7 -> 117.3 mm
- net Button3: track 115.6 -> 106.3 mm
- net Button1: track 129.0 -> 120.0 mm
- net Net-(D24-A): track 13.0 -> 21.7 mm
- net +5V_Isolated: track 285.6 -> 291.6 mm, vias 1 -> 2
- net DC_200V: track 33.9 -> 28.0 mm
- net I_meas: track 264.0 -> 258.2 mm
- net Net-(U12-VI): track 31.1 -> 27.0 mm
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Other:
- board size 250 x 135.5 mm -> 219 x 135.5 mm
