File: [02]Designs/KiCad Design/463 term project.kicad_pcb (KiCad board)
At the start: 2 copper layers, 219 x 135.5 mm, 141 parts, among them J1 Conn_01x02_Pin, J10 Conn_01x01_Pin, J11 Conn_01x01_Pin, J12 Conn_01x01_Pin, J13 Conn_01x01_Pin, J14 Conn_01x01_Pin, J15 Conn_01x01_Pin, J16 Conn_01x01_Pin, J17 Conn_01x01_Pin, J18 Conn_01x02_Pin, J19 Conn_01x02_Pin, J2 Screw_Terminal_01x01, J20 Conn_01x02_Pin, J21 Conn_01x02_Pin, J22 Conn_01x02_Pin, J23 Conn_01x02_Pin, J24 Conn_01x02_Pin, J25 Conn_01x02_Pin, J26 Conn_01x02_Pin, J3 Screw_Terminal_01x01, J4 Conn_01x03_Pin, J5 Screw_Terminal_01x01, J6 Screw_Terminal_01x01, J7 Conn_01x02_Pin, J8 Conn_01x01_Pin, J9 Conn_01x01_Pin, Q1 BC547, Q10 PJMH099N60EC, Q11 PJMH099N60EC, Q2 BC547, Q7 PJMH099N60EC, Q8 PJMH099N60EC, Q9 PJMH099N60EC, SW1 SW_Nidec_CAS-120A1, T2 Transformer, U1 6N135, U10 ADuM1200AR, U11 IR2110, U12 LM7805_TO220, U14 LM7815_TO220, U16 LD1117S33TR_SOT223, U17 LD1117S33TR_SOT223, U18 5 Button Module, U19 LM7812_TO220, U2 6N135, U20 LM7812_TO220, U3 74HC00, U4 IR2110, U5 IR2110, U6 ACS712xLCTR-30A, U8 ADuM1200AR, U9 ADuM1200AR

Commit message: Minor PCB Shematic Correction & File Arrangements
Parts:
- J4: value Conn_01x03_Pin -> Speed Measurement Sensor Connector
Changed lines of the file:
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@@
 			)
 		)
-		(property "Value" "Conn_01x03_Pin"
+		(property "Value" "Speed Measurement Sensor Connector"
 			(at 0 7.41 0)
 			(layer "F.Fab")

Commit message: Schematic Update & New Software Update (LED and Buttons Added)
Connections:
- R28 pad 1: /LED -> /LED_brake
- R32 pad 1: /LED_brake -> /LED
- U7 pad 36: /LED_brake -> /LED
- U7 pad 37: /LED -> /LED_brake
Routing:
- net /LED_brake: track 5.15 -> 2.88 mm
- net /LED: track 2.88 -> 5.15 mm
Changed lines of the file:
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@@
 			(size 0.8 0.8)
 			(layers "F.Cu" "F.Mask" "F.Paste")
-			(net 97 "/LED_brake")
+			(net 48 "/LED")
 			(pintype "passive")
 			(solder_mask_margin 0.1)
@@
 			(size 0.8 0.8)
 			(layers "F.Cu" "F.Mask" "F.Paste")
-			(net 48 "/LED")
+			(net 97 "/LED_brake")
 			(pintype "passive")
 			(solder_mask_margin 0.1)
@@
 			(layers "*.Cu" "*.Mask")
 			(remove_unused_layers no)
-			(net 97 "/LED_brake")
+			(net 48 "/LED")
 			(pinfunction "IO22")
 			(pintype "bidirectional")
@@
 			(layers "*.Cu" "*.Mask")
 			(remove_unused_layers no)
-			(net 48 "/LED")
+			(net 97 "/LED_brake")
 			(pinfunction "IO23")
 			(pintype "bidirectional")
@@
 	)
 	(segment
-		(start 233.75 156.26)
-		(end 233.65 156.16)
+		(start 228.3 157.75)
+		(end 229.52 157.75)
 		(width 0.5)
 		(layer "F.Cu")
@@
 	)
 	(segment
-		(start 233.75 159)
-		(end 233.75 156.26)
+		(start 229.52 157.75)
+		(end 231.11 156.16)
+		(width 0.5)
+		(layer "F.Cu")
+		(net 48)
+	)
+	(segment
+		(start 227.25 159)
+		(end 227.25 158.8)
+		(width 0.5)
+		(layer "F.Cu")
+		(net 48)
+	)
+	(segment
+		(start 227.25 158.8)
+		(end 228.3 157.75)
 		(width 0.5)
 		(layer "F.Cu")
@@
 	)
 	(segment
-		(start 228.3 157.75)
-		(end 229.52 157.75)
-		(width 0.5)
-		(layer "F.Cu")
-		(net 97)
-	)
-	(segment
-		(start 229.52 157.75)
-		(end 231.11 156.16)
-		(width 0.5)
-		(layer "F.Cu")
-		(net 97)
-	)
-	(segment
-		(start 227.25 159)
-		(end 227.25 158.8)
+		(start 233.75 156.26)
+		(end 233.65 156.16)
 		(width 0.5)
 		(layer "F.Cu")
@@
 	)
 	(segment
-		(start 227.25 158.8)
-		(end 228.3 157.75)
+		(start 233.75 159)
+		(end 233.75 156.26)
 		(width 0.5)
 		(layer "F.Cu")
